File: HRTIM_CHC2_HRTIM_CHD1.kicad_sch (KiCad schematic)
At the start: 9 parts, among them U13 STSPIN240

Commit message: Add files via upload
Parts:
- added TP28: "HRTCHC2_P", TestPoint:TestPoint_Pad_1.0x1.0mm, symbol Connector:TestPoint
- added TP29: "HRTCHC2", TestPoint:TestPoint_Pad_1.0x1.0mm, symbol Connector:TestPoint
- added TP30: "HRTCHC2_O1", TestPoint:TestPoint_Pad_1.0x1.0mm, symbol Connector:TestPoint
- added TP31: "HRTCHC2_O2", TestPoint:TestPoint_Pad_1.0x1.0mm, symbol Connector:TestPoint
- added TP32: "HRTCHD1_P", TestPoint:TestPoint_Pad_1.0x1.0mm, symbol Connector:TestPoint
- added TP33: "HRTCHD1", TestPoint:TestPoint_Pad_1.0x1.0mm, symbol Connector:TestPoint
- added TP34: "HRTCHD1_O1", TestPoint:TestPoint_Pad_1.0x1.0mm, symbol Connector:TestPoint
- added TP35: "HRTCHD1_O2", TestPoint:TestPoint_Pad_1.0x1.0mm, symbol Connector:TestPoint
Connections:
- net HRTIM_CHC2: now also TP29.1
- net HRTIM_CHC2_OUT1: now also TP30.1
- net HRTIM_CHC2_OUT2: now also TP31.1
- net HRTIM_CHC2_PHASE: now also TP28.1
- net HRTIM_CHD1: now also TP33.1
- net HRTIM_CHD1_OUT1: now also TP34.1
- net HRTIM_CHD1_OUT2: now also TP35.1
- net HRTIM_CHD1_PHASE: now also TP32.1
- net EN renamed EN_U13
Other:
- moved on the sheet: C60, C61, C62, R50, R51, R52, R53, R54, U13
