File: TIM1_CH4_TIM12_CH2.kicad_sch (KiCad schematic)
At the start: 9 parts, among them U16 STSPIN240

Commit message: Add files via upload
Parts:
- added TP18: "T1CH4_P", TestPoint:TestPoint_Pad_1.0x1.0mm, symbol Connector:TestPoint
- added TP19: "T1CH4", TestPoint:TestPoint_Pad_1.0x1.0mm, symbol Connector:TestPoint
- added TP20: "T1CH4_O1", TestPoint:TestPoint_Pad_1.0x1.0mm, symbol Connector:TestPoint
- added TP21: "T1CH4_O2", TestPoint:TestPoint_Pad_1.0x1.0mm, symbol Connector:TestPoint
- added TP22: "T12CH2_P", TestPoint:TestPoint_Pad_1.0x1.0mm, symbol Connector:TestPoint
- added TP23: "T12CH2", TestPoint:TestPoint_Pad_1.0x1.0mm, symbol Connector:TestPoint
- added TP24: "T12CH2_O1", TestPoint:TestPoint_Pad_1.0x1.0mm, symbol Connector:TestPoint
- added TP25: "T12CH2_O2", TestPoint:TestPoint_Pad_1.0x1.0mm, symbol Connector:TestPoint
Connections:
- net TIM12_CH2: now also TP23.1
- net TIM12_CH2_OUT1: now also TP24.1
- net TIM12_CH2_OUT2: now also TP25.1
- net TIM12_CH2_PHASE: now also TP22.1
- net TIM1_CH4: now also TP19.1
- net TIM1_CH4_OUT1: now also TP20.1
- net TIM1_CH4_OUT2: now also TP21.1
- net TIM1_CH4_PHASE: now also TP18.1
- net EN renamed EN_U16
Other:
- moved on the sheet: C69, C70, C71, R65, R66, R67, R68, R69, U16
