File: eddy_current_sensors.kicad_sch (KiCad schematic)
At the start: 15 parts, among them J4 DB25_Receptacle_MountingHoles, U10 LDC1614, U9 LDC1614

Commit message: Add files via upload
Parts:
- added TP26: "SDA", TestPoint:TestPoint_THTPad_D1.0mm_Drill0.5mm, symbol Connector:TestPoint
- added TP27: "SCL", TestPoint:TestPoint_THTPad_D1.0mm_Drill0.5mm, symbol Connector:TestPoint
Connections:
- net I2C4_SCL: now also TP27.1
- net I2C4_SDA: now also TP26.1
- net SD: no longer R34.1, U10.6 (SD)
- new net: R34.1, U10.6 (SD)
- no-connect marks 0 -> 9
Other:
- moved on the sheet: J4, R34

Commit message: Add files via upload
Other:
- note removed: "DO WE NEED RESONATING CAPS ACROSS THE 2 INDUCTOR PINS?????? Need to check coil with impedance analyzer"
Changed lines of the file:
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@@
-		)
-	)
-	(text "DO WE NEED RESONATING CAPS ACROSS THE 2 INDUCTOR PINS??????\n\nNeed to check coil with impedance analyzer"
-		(exclude_from_sim no)
-		(at 167.386 170.688 0)
-		(effects
-			(font
-				(size 5 5)
-			)
 		)
 	)

Commit message: Add files via upload
Other:
- note added: "LDC 0 Sensors 0-3"
- note added: "LDC 1 Sensors 4-7"
- note removed: "LDC1614 Sensors 0-3"
- note removed: "LDC1614 Sensors 4-7"
Changed lines of the file:
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@@
 		)
 	)
-	(text "LDC1614\nSensors 0-3"
+	(text "LDC 0\nSensors 0-3"
 		(exclude_from_sim no)
 		(at 38.354 42.418 0)
@@
 		)
 	)
-	(text "LDC1614\nSensors 4-7"
+	(text "LDC 1\nSensors 4-7"
 		(exclude_from_sim no)
 		(at 185.42 42.418 0)
