File: kasm_pcb_rev2.kicad_pcb (KiCad board)
At the start: 6 copper layers, 121.2 x 70.6 mm, 232 parts, among them J1 Conn_01x02, J2 Conn_01x02, J20 09564527612, J3 Conn_01x06, J4 DB25_Receptacle_MountingHoles, J5 Conn_01x06, J6 Conn_01x06, J7 Conn_01x03, SW1 SW_Push, SW2 SW_Push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

Commit message: Add files via upload
Parts:
- added C33: 100nF, Capacitor_SMD:C_0402_1005Metric, F.Cu at (137.9, 60.2)
- added D3: LED_RED, LED_SMD:LED_0603_1608Metric, F.Cu at (133.7, 58.8)
- added D4: LED_RED, LED_SMD:LED_0603_1608Metric, F.Cu at (133.7, 57.0)
- added D5: LED_GREEN, LED_SMD:LED_0603_1608Metric, F.Cu at (120.5, 80.1)
- added D6: LED_WHITE, LED_SMD:LED_0402_1005Metric, F.Cu at (102.0, 87.8)
- added D7: LED_WHITE, LED_SMD:LED_0402_1005Metric, F.Cu at (103.1, 87.8)
- added D8: LED_WHITE, LED_SMD:LED_0402_1005Metric, F.Cu at (104.3, 87.8)
- added G***: LOGO, LOGO, B.Cu at (129.8, 69.6)
- added R15: 1k, Resistor_SMD:R_0402_1005Metric, F.Cu at (131.1, 58.5)
- added R17: 1k, Resistor_SMD:R_0402_1005Metric, F.Cu at (131.1, 57.3)
- added R18: 100, Resistor_SMD:R_0402_1005Metric, F.Cu at (120.2, 81.6)
- added R19: 100, Resistor_SMD:R_0402_1005Metric, F.Cu at (102.0, 90.0)
- added R20: 100, Resistor_SMD:R_0402_1005Metric, F.Cu at (103.1, 90.0)
- added R21: 100, Resistor_SMD:R_0402_1005Metric, F.Cu at (104.3, 90.0)
- added R22: 49.9, Resistor_SMD:R_0402_1005Metric, F.Cu at (95.7, 83.9)
- added TP18: "T1CH4_P", TestPoint:TestPoint_Pad_1.0x1.0mm, F.Cu at (145.1, 61.9)
- added TP19: "T1CH4", TestPoint:TestPoint_Pad_1.0x1.0mm, F.Cu at (139.2, 68.0)
- added TP20: "T1CH4_O1", TestPoint:TestPoint_Pad_1.0x1.0mm, F.Cu at (145.7, 58.0)
- added TP21: "T1CH4_O2", TestPoint:TestPoint_Pad_1.0x1.0mm, F.Cu at (148.3, 58.0)
- added TP22: "T12CH2_P", TestPoint:TestPoint_Pad_1.0x1.0mm, F.Cu at (139.2, 64.3)
- added TP23: "T12CH2", TestPoint:TestPoint_Pad_1.0x1.0mm, F.Cu at (141.6, 61.9)
- added TP24: "T12CH2_O1", TestPoint:TestPoint_Pad_1.0x1.0mm, F.Cu at (151.6, 58.0)
- added TP25: "T12CH2_O2", TestPoint:TestPoint_Pad_1.0x1.0mm, F.Cu at (155.0, 58.0)
- added TP26: "SDA", TestPoint:TestPoint_THTPad_D1.0mm_Drill0.5mm, F.Cu at (93.1, 67.8)
- added TP27: "SCL", TestPoint:TestPoint_THTPad_D1.0mm_Drill0.5mm, F.Cu at (93.1, 64.0)
- added TP28: "HRTCHC2_P", TestPoint:TestPoint_Pad_1.0x1.0mm, F.Cu at (154.4, 62.6)
- added TP29: "HRTCHC2", TestPoint:TestPoint_Pad_1.0x1.0mm, F.Cu at (158.8, 62.6)
- added TP30: "HRTCHC2_O1", TestPoint:TestPoint_Pad_1.0x1.0mm, F.Cu at (153.4, 70.7)
- added TP31: "HRTCHC2_O2", TestPoint:TestPoint_Pad_1.0x1.0mm, F.Cu at (157.9, 70.7)
- added TP32: "HRTCHD1_P", TestPoint:TestPoint_Pad_1.0x1.0mm, F.Cu at (156.5, 62.6)
- added TP33: "HRTCHD1", TestPoint:TestPoint_Pad_1.0x1.0mm, F.Cu at (160.5, 60.5)
- added TP34: "HRTCHD1_O1", TestPoint:TestPoint_Pad_1.0x1.0mm, F.Cu at (164.2, 71.9)
- added TP35: "HRTCHD1_O2", TestPoint:TestPoint_Pad_1.0x1.0mm, F.Cu at (161.2, 71.9)
- added U6: 74LVC2G07, Package_TO_SOT_SMD:SOT-23-6, F.Cu at (137.8, 57.8)
- moved C31 9.45 mm to (94.5, 74.7), turned to 90 degrees
- moved J5 8.90 mm to (120.8, 56.8), turned to -90 degrees
- moved L3 3.60 mm to (92.1, 82.0), turned to 0 degrees
- moved C26 3.42 mm to (102.1, 59.7)
- moved U3 3.42 mm to (98.7, 59.6)
- moved R33 3.34 mm to (163.7, 58.4)
- moved R32 3.34 mm to (163.7, 57.4)
- moved C42 3.29 mm to (165.7, 57.4)
- moved TP6 1.70 mm to (142.2, 113.9)
- moved TP4 1.70 mm to (139.7, 114.9)
- moved TP2 1.69 mm to (137.1, 113.9)
- moved TP3 1.69 mm to (134.6, 114.6)
- moved TP16 1.69 mm to (144.7, 114.9)
- moved J6 1.11 mm to (134.5, 119.0)
- moved TP14 1.09 mm to (83.1, 78.9)
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Connections:
- net /Actuators/HRTIM_CHC2_HRTIM_CHD1/EN renamed EN_U13
- net /Actuators/TIM1_CH4_TIM12_CH2/EN renamed EN_U16
- J20 pad MH1: unconnected-(J20-PadMH1) -> GND
- J20 pad MH2: unconnected-(J20-PadMH2) -> GND
- R34 pad 1: /Eddy Current Sensors/SD -> Net-(U10-SD)
- U10 pad 6: /Eddy Current Sensors/SD -> Net-(U10-SD)
- U5 pad 15: ADC2_INP10 -> unconnected-(U5-PC0-Pad15)
- U5 pad 17: LDC0_INTB -> unconnected-(U5-PC2_C-Pad17)
- U5 pad 18: LDC1_INTB -> unconnected-(U5-PC3_C-Pad18)
- U5 pad 25: TIM2_CH4_LDC -> Net-(U5-PA3)
- U5 pad 32: ADC1_INP4 -> LDC0_INTB
- U5 pad 33: unconnected-(U5-PC5-Pad33) -> LDC1_INTB
- U5 pad 34: ADC2_INP9 -> LED0
- U5 pad 35: ADC1_INP5 -> LED1
- U5 pad 36: SPI6_MUX_S -> LED2
- U5 pad 52: SPI6_MUX_~{OE} -> unconnected-(U5-PB13-Pad52)
Routing:
- net REF: track 0.00 -> 207.6 mm, vias 0 -> 15
- net SPI6_MOSI: track 0.00 -> 138.5 mm, vias 0 -> 3
- net SPI6_MISO: track 0.00 -> 131.8 mm, vias 0 -> 3
- net TIM16_CH1_PHASE: track 0.00 -> 130.6 mm, vias 0 -> 6
- net TIM16_CH1: track 0.00 -> 127.2 mm, vias 0 -> 6
- net TIM1_CH3_PHASE: track 0.00 -> 112.2 mm, vias 0 -> 4
- net HRTIM_CHB2_PHASE: track 0.00 -> 109.5 mm, vias 0 -> 4
- net SPI6_SCK: track 0.00 -> 109.3 mm, vias 0 -> 3
- net TIM4_CH2: track 0.00 -> 105.7 mm, vias 0 -> 4
- net SPI6_NSS: track 0.00 -> 101.5 mm, vias 0 -> 3
- net TIM1_CH2_PHASE: track 0.00 -> 100.0 mm, vias 0 -> 4
- net I2C4_SCL: track 1.50 -> 99.5 mm, vias 0 -> 7
- net TIM13_CH1: track 0.00 -> 95.5 mm, vias 0 -> 4
- net TIM13_CH1_PHASE: track 0.00 -> 91.1 mm, vias 0 -> 4
- net I2C4_SDA: track 2.88 -> 91.0 mm, vias 0 -> 5
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Other:
- board size 121.2 x 70.6 mm -> 121 x 70.6 mm
- board text added: "0"
- board text added: "1"
- board text added: "1.8V PWR BAD"
- board text added: "2"
- board text added: "3.3V"
- board text added: "3.3V POWER"
- board text added: "Actuators"
- board text added: "All design files at github.com/gabeak2/KASM_ACTUATOR_PCB_REV2"
- board text added: "BOOT0"
- board text added: "KASM/UH88 ACTUATOR PCBA REV2"
- board text added: "LDCs"
- board text added: "PROG"
- board text added: "RESET"
- board text added: "RX"
- board text added: "S/N:"
- board text added: "SCL"
- board text added: "SDA"
- board text added: "SPI2"
- board text added: "SWCLK"
- board text added: "SWDIO"
- board text added: "SWO"
- board text added: "TX"
- board text added: "U13 FAULT"
- board text added: "U16 FAULT"
- board text added: "UART4"
- board text added: "~{RST}"

Commit message: Add files via upload
Parts:
- added D9: LED_GREEN, LED_SMD:LED_0603_1608Metric, F.Cu at (132.7, 113.9)
- added R23: 220, Resistor_SMD:R_0402_1005Metric, F.Cu at (132.4, 117.3)
- R19, R20, R21: value 100 -> 220
- moved TP16 0.60 mm to (144.7, 115.5)
- moved TP2 0.60 mm to (137.1, 114.5)
- moved TP3 0.60 mm to (134.6, 115.2)
- moved TP4 0.60 mm to (139.7, 115.5)
- moved TP6 0.60 mm to (142.2, 114.5)
Routing:
- net Net-(D9-K): track 0.00 -> 2.22 mm
- net SPI6_NSS: track 101.5 -> 103.3 mm
- net +3.3V: track 14.6 -> 16.0 mm, vias 46 -> 47
- net /Eddy Current Sensors/IN4B: track 24.9 -> 25.6 mm
- net SPI6_MOSI: track 138.5 -> 137.9 mm
- net SPI6_MISO: track 131.8 -> 131.2 mm
- net SPI6_SCK: track 109.3 -> 108.7 mm
- net GND: vias 182 -> 183
Other:
- board text added: "+1.8V"
- board text added: "+12V"
- board text added: "+3.3V"
- board text removed: "12V"
