File: mcu.kicad_sch (KiCad schematic)
At the start: 42 parts, among them J3 Conn_01x06, J5 Conn_01x06, J6 Conn_01x06, J7 Conn_01x03, SW1 SW_Push, SW2 SW_Push, U3 M24C02-WMN, U5 STM32H750VBTx, Y1 24MHz, 9pF

Commit message: Add files via upload
Parts:
- added D6, D7, D8: LED_WHITE, LED_SMD:LED_0402_1005Metric, symbol Device:LED
- added R19, R20, R21: 100, Resistor_SMD:R_0402_1005Metric, symbol Device:R_US
- added R22: 49.9, Resistor_SMD:R_0402_1005Metric, symbol Device:R_Small_US
Connections:
- net ADC1_INP4 is gone; now on net LDC0_INTB: U5.32 (PC4)
- net GND: now also R19.2, R20.2, R21.2
- net LDC0_INTB: no longer U5.17 (PC2_C)
- net LDC1_INTB: now also U5.33 (PC5); no longer U5.18 (PC3_C)
- net TIM2_CH4_LDC: now also R22.2; no longer U5.25 (PA3)
- net ADC1_INP5 renamed LED1
- net LED1: now also D7.2 (A)
- net ADC2_INP10: no longer names the net of U5.15 (PC0)
- net ADC2_INP9 renamed LED0
- net LED0: now also D6.2 (A)
- net SPI6_MUX_S renamed LED2
- net LED2: now also D8.2 (A)
- net SPI6_MUX_~{OE}: no longer names the net of U5.52 (PB13)
- new net: R22.1, U5.25 (PA3)
- new net: D8.1 (K), R21.1
- new net: D7.1 (K), R20.1
- new net: D6.1 (K), R19.1
- no-connect marks 6 -> 9
Other:
- note added: "LED INDICATORS"
- moved on the sheet: J3, J5, J6, J7, TP10, TP11, TP14, TP15, TP16, TP17, TP2, TP3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

Commit message: Add files via upload
Parts:
- added D9: LED_GREEN, LED_SMD:LED_0603_1608Metric, symbol Device:LED
- added R23: 220, Resistor_SMD:R_0402_1005Metric, symbol Device:R_US
- R19, R20, R21: value 100 -> 220; LCSC C98836 -> C25091
Connections:
- net +3.3V: now also D9.2 (A)
- net SPI6_NSS: now also R23.2
- new net: D9.1 (K), R23.1
Other:
- note added: "Series Terminated ~50-Ohm trace"
- moved on the sheet: D6, D7, D8, R19, R20, R21

Commit message: Add files via upload
Parts:
- L3: value 100uH -> 10uH
Changed lines of the file:
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@@
 			)
 		)
-		(property "Value" "100uH"
+		(property "Value" "10uH"
 			(at 182.88 70.2911 90)
 			(effects
