File: power.kicad_sch (KiCad schematic)
At the start: 54 parts, among them J1 Conn_01x02, J2 Conn_01x02, U1 TPS5430DDA, U2 TPS54620

Commit message: Add files via upload
Parts:
- added D5: LED_GREEN, LED_SMD:LED_0603_1608Metric, symbol Device:LED
- added R18: 100, Resistor_SMD:R_0402_1005Metric, symbol Device:R_US
Connections:
- net +3.3V: now also D5.2 (A)
- net GND: now also R18.2
- new net: D5.1 (K), R18.1

Commit message: Add files via upload
Other:
- note added: "Rt = 240k --> ~200kHz switching frequency"
- moved on the sheet: C1, C10, C11, C12, C13, C14, C15, C16, C17, C18, C19, C2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

Commit message: Add files via upload
Parts:
- R18: LCSC C98836 -> C106232
Changed lines of the file:
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@@
 			)
 		)
-		(property "LCSC" "C98836"
+		(property "LCSC" "C106232"
 			(at 314.96 78.74 0)
 			(effects
